Commit message: Gazebo sim

File: description/urdf/embla.gazebo.xacro (robot description, xacro)
@@ -1,12 +1,15 @@
 <?xml version="1.0"?>
+<!--
+	This macro contains _common_ Gazebo tags.
+	Gazebo information for individual wheels are defined in the wheel.xacro file.
+	Material colors are defined near the respective links.
+-->
 <robot xmlns:xacro="http://www.ros.org/wiki/xacro" name="embla">
-	<gazebo reference="base_link">
-		<material>Gazebo/Green</material>
-	</gazebo>
-	<gazebo reference="spacer">
-		<material>Gazebo/lightGrey</material>
-	</gazebo>
 	<gazebo>
-		<plugin name="gazebo_ros_control" filename="libgazebo_ros_control.so"/>
+		<plugin filename="libgazebo_ros2_control.so" name="gazebo_ros2_control">
+			<robot_param>robot_description</robot_param>
+			<robot_param_node>robot_state_publisher</robot_param_node>
+			<parameters></parameters>
+		</plugin>
 	</gazebo>
 </robot>

File: description/urdf/embla_description.urdf.xacro (robot description, xacro)
@@ -109,5 +109,6 @@
 		</visual>
 		<visual name="spacer">
-			<origin xyz="${-chassisLength/2 + 0.0035} ${-chassisWidth/2 + 0.016} -0.0165" rpy="0 0 0" />
+			<origin xyz="${-chassisLength/2 + 0.0035} ${-chassisWidth/2 + 0.016} -0.0165"
+				rpy="0 0 0" />
 			<geometry>
 				<cylinder length="0.03" radius="0.0025" />
@@ -118,13 +119,20 @@
 			<origin xyz="0 0 0" rpy="0 0 0" />
 			<mass value="${chassisMass}" />
-			<xacro:box_inertia m="${chassisMass}" x="${chassisLength}" y="${chassisWidth}" z="${chassisHeight}" />
+			<xacro:box_inertia m="${chassisMass}" x="${chassisLength}" y="${chassisWidth}"
+				z="${chassisHeight}" />
 		</inertial>
 	</link>
+	<gazebo reference="base_link">
+		<material>Gazebo/Green</material>
+	</gazebo>
+	<gazebo reference="spacer">
+		<material>Gazebo/lightGrey</material>
+	</gazebo>
 	<!-- Add wheels -->
 	<xacro:include filename="wheel.xacro" />
-	<xacro:wheel lr="left" fr="front" tY="1" tX="1"/>
-	<xacro:wheel lr="right" fr="front" tY="-1" tX="1"/>
-	<xacro:wheel lr="left" fr="rear" tY="1" tX="-1"/>
-	<xacro:wheel lr="right" fr="rear" tY="-1" tX="-1"/>
+	<xacro:wheel lr="left" fr="front" tY="1" tX="1" />
+	<xacro:wheel lr="right" fr="front" tY="-1" tX="1" />
+	<xacro:wheel lr="left" fr="rear" tY="1" tX="-1" />
+	<xacro:wheel lr="right" fr="rear" tY="-1" tX="-1" />
 	<!-- Lidar -->
 	<xacro:include filename="lidar.xacro" />

File: description/urdf/wheel.xacro (robot description, xacro)
@@ -45,15 +45,22 @@
 			</inertial>
 		</link>
+		<!-- Gazebo sim -->
 		<gazebo reference="${lr}_${fr}_wheel">
 			<material>Gazebo/FlatBlack</material>
+			<mu1>100000000000000.0</mu1>
+			<mu2>1000000000.0</mu2>
+			<kp>1000000000000.0</kp>
+			<kd>10.0</kd>
+			<minDepth>0.001</minDepth>
+			<maxVel>0.1</maxVel>
+			<fdir1>1 0 0</fdir1>
 		</gazebo>
 		<transmission name="${lr}_${fr}_trans">
 			<type>transmission_interface/SimpleTransmission</type>
-			<joint name="${lr}_${fr}_wheel_joint">
+			<joint name="${lr}_${fr}_wheel_joint" role="joint_${lr}_${fr}">
 				<hardwareInterface>hardware_interface/VelocityJointInterface</hardwareInterface>
+				<mechanicalReduction>1</mechanicalReduction>
 			</joint>
-			<actuator name="${lr}_${fr}_motor">
-				<mechanicalReduction>1</mechanicalReduction>
-			</actuator>
+			<actuator name="${lr}_${fr}_motor" role="actuator_${lr}_${fr}" />
 		</transmission>
 	</xacro:macro>
