Commit message: Launch file fixes

File: description/urdf/lidar.xacro (robot description, xacro)
@@ -36,4 +36,12 @@
 		</inertial>
 	</link>
+	<!-- laser_frame is coindicent with lidar_link and is just used for compatibility with
+	components expecting laser_frame -->
+	<link name="laser_frame" />
+	<joint name="laser_frame_joint" type="fixed">
+		<parent link="lidar_link" />
+		<child link="laser_frame" />
+		<origin xyz="0 0 0" />
+	</joint>
 	<!-- from ROSbot 2.0
 	https://github.com/husarion/rosbot_description/blob/master/src/rosbot_description/urdf/rosbot.xacro -->

Commit message: Launch file fixes: - set angle_compensate: true for lidar - fixed setting params file for slam_toolbox - delayed launch of slam_toolbox after joint_state_publisher - also removed laser_frame, now uses lidar_link

File: description/urdf/lidar.xacro (robot description, xacro)
@@ -11,6 +11,5 @@
 			Origin is at center of Lidar which is placed on chassis top, 5 cm forward of midpoint.
 			NOTE The origin has been rotated PI radians around Z because the RPLidar has X pointing backwards
-		and Y pointing right compared to conventional robot orientation (X forward, Y left, Z up).
-			This, however, will mess up the /scan data when running in Gazebo. -->
+		and Y pointing right compared to conventional robot orientation (X forward, Y left, Z up). -->
 		<origin xyz="0.04 0 ${chassisHeight/2 + lidarHeight/2}" rpy="0 0 ${PI}" />
 	</joint>
@@ -36,12 +35,4 @@
 		</inertial>
 	</link>
-	<!-- laser_frame is coindicent with lidar_link and is just used for compatibility with
-	components expecting laser_frame -->
-	<link name="laser_frame" />
-	<joint name="laser_frame_joint" type="fixed">
-		<parent link="lidar_link" />
-		<child link="laser_frame" />
-		<origin xyz="0 0 0" />
-	</joint>
 	<!-- from ROSbot 2.0
 	https://github.com/husarion/rosbot_description/blob/master/src/rosbot_description/urdf/rosbot.xacro -->
