Commit message: Fix URDF: Colons in comments can mess up passing the robot_description on command line

File: description/urdf/imu.xacro (robot description, xacro)
@@ -34,5 +34,5 @@
 		<material>Gazebo/Orange</material>
 	</gazebo>
-	<!-- Team Hector's IMU plugin: https://github.com/tu-darmstadt-ros-pkg/hector_gazebo -->
+	<!-- Team Hector's IMU plugin https://github.com/tu-darmstadt-ros-pkg/hector_gazebo -->
 	<gazebo>
 		<plugin name="imu_controller" filename="libhector_gazebo_ros_imu.so">

File: description/urdf/lidar.xacro (robot description, xacro)
@@ -10,5 +10,5 @@
 		<!--
 			Origin is at center of Lidar which is placed on chassis top, 5 cm forward of midpoint.
-			NOTE: The origin has been rotated PI radians around Z because the RPLidar has X pointing backwards and Y pointing right compared to conventional robot orientation (X forward, Y left, Z up).
+			NOTE The origin has been rotated PI radians around Z because the RPLidar has X pointing backwards and Y pointing right compared to conventional robot orientation (X forward, Y left, Z up).
 			This, however, will mess up the /scan data when running in Gazebo. -->
 		<origin xyz="0.04 0 ${chassisHeight/2 + lidarHeight/2}" rpy="0 0 ${PI}" />
@@ -34,37 +34,37 @@
 		</inertial>
 	</link>
-	<!-- from ROSbot 2.0: https://github.com/husarion/rosbot_description/blob/master/src/rosbot_description/urdf/rosbot.xacro -->
-  <!-- RpLidar using GPU -->
-  <gazebo reference="lidar_link">
-    <sensor type="gpu_ray" name="head_rplidar_sensor">
-      <pose>0 0 0.06 0 0 0</pose>
-      <visualize>false</visualize>
-      <update_rate>40</update_rate>
-      <ray>
-        <scan>
-          <horizontal>
-            <samples>720</samples>
-            <resolution>1</resolution>
-            <min_angle>-${PI}</min_angle>
-            <max_angle>${PI}</max_angle>
-          </horizontal>
-        </scan>
-        <range>
-          <min>0.2</min>
-          <max>12.0</max>
-          <resolution>0.01</resolution>
-        </range>
-        <noise>
-          <type>gaussian</type>
-          <mean>0.0</mean>
-          <stddev>0.01</stddev>
-        </noise>
-      </ray>
-      <plugin name="gazebo_ros_head_rplidar_controller" filename="libgazebo_ros_gpu_laser.so">
-        <topicName>scan</topicName>
-        <frameName>lidar_link</frameName>
-      </plugin>
-    </sensor>
-	<material>Gazebo/Black</material>
-  </gazebo>
+	<!-- from ROSbot 2.0 https://github.com/husarion/rosbot_description/blob/master/src/rosbot_description/urdf/rosbot.xacro -->
+	<!-- RpLidar using GPU -->
+	<gazebo reference="lidar_link">
+		<sensor type="gpu_ray" name="head_rplidar_sensor">
+			<pose>0 0 0.06 0 0 0</pose>
+			<visualize>false</visualize>
+			<update_rate>40</update_rate>
+			<ray>
+				<scan>
+					<horizontal>
+						<samples>720</samples>
+						<resolution>1</resolution>
+						<min_angle>-${PI}</min_angle>
+						<max_angle>${PI}</max_angle>
+					</horizontal>
+				</scan>
+				<range>
+					<min>0.2</min>
+					<max>12.0</max>
+					<resolution>0.01</resolution>
+				</range>
+				<noise>
+					<type>gaussian</type>
+					<mean>0.0</mean>
+					<stddev>0.01</stddev>
+				</noise>
+			</ray>
+			<plugin name="gazebo_ros_head_rplidar_controller" filename="libgazebo_ros_gpu_laser.so">
+				<topicName>scan</topicName>
+				<frameName>lidar_link</frameName>
+			</plugin>
+		</sensor>
+		<material>Gazebo/Black</material>
+	</gazebo>
 </robot>

Commit message: Loc. launch files and rotated IMU

File: description/urdf/imu.xacro (robot description, xacro)
@@ -9,5 +9,5 @@
 		<child link="imu_link" />
 		<!-- Origin is at center of IMU which is placed on chassis top, a little back from midpoint -->
-		<origin xyz="-0.05 0 ${chassisHeight/2 + imuHeight/2}" rpy="0 0 ${PI/2}" />
+		<origin xyz="-0.05 0 ${chassisHeight/2 + imuHeight/2}" rpy="0 0 0" />
 	</joint>
 	<link name="imu_link">
