Commit message: WiP: Four wheel control

File: description/ros2_control/embla.ros2_control.xacro (robot description, xacro)
@@ -8,10 +8,10 @@
                 <param name="roboclaw_address">128</param>
             </hardware>
-            <joint name="${prefix}left_wheel_joint">
+            <joint name="${prefix}left_front_wheel_joint">
                 <command_interface name="velocity" />
                 <state_interface name="position" />
                 <state_interface name="velocity" />
             </joint>
-            <joint name="${prefix}right_wheel_joint">
+            <joint name="${prefix}right_front_wheel_joint">
                 <command_interface name="velocity" />
                 <state_interface name="position" />

Commit message: Work on four wheel drive

File: description/ros2_control/embla.ros2_control.xacro (robot description, xacro)
@@ -18,4 +18,14 @@
                 <state_interface name="velocity" />
             </joint>
+            <joint name="${prefix}left_rear_wheel_joint">
+                <command_interface name="velocity" />
+                <state_interface name="position" />
+                <state_interface name="velocity" />
+            </joint>
+            <joint name="${prefix}right_rear_wheel_joint">
+                <command_interface name="velocity" />
+                <state_interface name="position" />
+                <state_interface name="velocity" />
+            </joint>
         </ros2_control>
     </xacro:macro>

File: description/urdf/embla_description.urdf.xacro (robot description, xacro)
@@ -127,24 +127,4 @@
 	<xacro:wheel lr="left" fr="rear" tY="1" tX="-1"/>
 	<xacro:wheel lr="right" fr="rear" tY="-1" tX="-1"/>
-	<!--
-	-->
-	<!--
-	<joint name="left_wheel_joint" type="continuous">
-		<parent link="base_link"/>
-		<child link="left_front_wheel"/>
-		<origin xyz="${0.5 * wheelXDistance/2} ${1 * wheelYDistance/2} ${-chassisHeight/2 - (chassisGroundClearance - wheelRadius)}"/>
-		<axis xyz="0 1 0"/>
-		<dynamics damping="0.2"/>
-		<limit effort="100" velocity="1.0"/>
-	</joint>
-	<joint name="right_wheel_joint" type="continuous">
-		<parent link="base_link"/>
-		<child link="right_front_wheel"/>
-		<origin xyz="${0.5 * wheelXDistance/2} ${-1 * wheelYDistance/2} ${-chassisHeight/2 - (chassisGroundClearance - wheelRadius)}"/>
-		<axis xyz="0 1 0"/>
-		<dynamics damping="0.2"/>
-		<limit effort="100" velocity="1.0"/>
-	</joint>
-	-->
 	<!-- Lidar -->
 	<xacro:include filename="lidar.xacro" />

Commit message: URDF cleanup

File: description/ros2_control/embla.ros2_control.xacro (robot description, xacro)
@@ -1,5 +1,5 @@
 <?xml version="1.0"?>
 <robot xmlns:xacro="http://www.ros.org/wiki/xacro">
-    <xacro:macro name="embla_ros2_control" params="name prefix">
+    <xacro:macro name="embla_ros2_control" params="name">
         <ros2_control name="${name}" type="system">
             <hardware>
@@ -8,20 +8,20 @@
                 <param name="roboclaw_address">128</param>
             </hardware>
-            <joint name="${prefix}left_front_wheel_joint">
+            <joint name="left_front_wheel_joint">
                 <command_interface name="velocity" />
                 <state_interface name="position" />
                 <state_interface name="velocity" />
             </joint>
-            <joint name="${prefix}right_front_wheel_joint">
+            <joint name="right_front_wheel_joint">
                 <command_interface name="velocity" />
                 <state_interface name="position" />
                 <state_interface name="velocity" />
             </joint>
-            <joint name="${prefix}left_rear_wheel_joint">
+            <joint name="left_rear_wheel_joint">
                 <command_interface name="velocity" />
                 <state_interface name="position" />
                 <state_interface name="velocity" />
             </joint>
-            <joint name="${prefix}right_rear_wheel_joint">
+            <joint name="right_rear_wheel_joint">
                 <command_interface name="velocity" />
                 <state_interface name="position" />

File: description/urdf/embla.urdf.xacro (robot description, xacro)
@@ -2,8 +2,10 @@
 <!-- Main URDF including controller info -->
 <robot xmlns:xacro="http://www.ros.org/wiki/xacro" name="embla_robot">
-  <xacro:arg name="prefix" default="" />
+  <!-- Base URDF -->
   <xacro:include filename="embla_description.urdf.xacro" />
   <!-- Import ros2_control description -->
   <xacro:include filename="$(find embla_controller)/ros2_control/embla.ros2_control.xacro" />
-  <xacro:embla_ros2_control name="Embla" prefix="$(arg prefix)" />
+  <xacro:embla_ros2_control name="Embla" />
+  <!-- Gazebo common -->
+  <xacro:include filename="embla.gazebo.xacro" />
 </robot>

File: description/urdf/embla_description.urdf.xacro (robot description, xacro)
@@ -1,23 +1,22 @@
 <?xml version="1.0"?>
-<robot name="embla"
-	xmlns:xacro="http://www.ros.org/wiki/xacro">
+<robot name="embla" xmlns:xacro="http://www.ros.org/wiki/xacro">
 	<xacro:property name="PI" value="3.1415926535897931" />
+	<!-- Chassis info -->
+	<!-- three 3 mm plates + 30 mm spacers between -->
 	<xacro:property name="chassisHeight" value="0.069" />
-	<!-- three 3 mm plates + 30 mm spacers between -->
 	<xacro:property name="chassisLength" value="0.17" />
 	<xacro:property name="chassisWidth" value="0.14" />
+	<!-- Total 1950 including 4 x 80 g wheels. Wheels' mass and inertia are specified for each wheel -->
 	<xacro:property name="chassisMass" value="1.630" />
-	<!-- Total 1950 including 4 x 80 g wheels. Wheels' mass and inertia are specified for each wheel -->
+	<!-- Distance to bottom of chassis -->
 	<xacro:property name="chassisGroundClearance" value="0.074" />
-	<!-- Distance to bottom of chassis -->
+	<!-- Wheel info -->
 	<xacro:property name="wheelWidth" value="0.04" />
 	<xacro:property name="wheelRadius" value="0.04" />
-	<!-- NB: Radius, not diameter! -->
 	<xacro:property name="wheelMass" value="0.08" />
+	<!-- Sideways distance between wheel centers -->
 	<xacro:property name="wheelYDistance" value="0.1875" />
-	<!-- Sideways distance between wheel centers -->
+	<!-- Front/back distance between wheel centers -->
 	<xacro:property name="wheelXDistance" value="0.1125" />
-	<!-- Front/back distance between wheel centers -->
-	<!-- <xacro:include filename="embla.gazebo.xacro" /> -->
 	<xacro:include filename="$(find embla_controller)/urdf/macros.xacro" />
 	<xacro:include filename="materials.xacro" />

Commit message: URDF

File: description/ros2_control/embla.ros2_control.xacro (robot description, xacro)
@@ -1,4 +1,4 @@
 <?xml version="1.0"?>
-<robot xmlns:xacro="http://www.ros.org/wiki/xacro">
+<robot name="embla" xmlns:xacro="http://www.ros.org/wiki/xacro">
     <xacro:macro name="embla_ros2_control" params="name">
         <ros2_control name="${name}" type="system">

File: description/urdf/embla.urdf.xacro (robot description, xacro)
@@ -1,9 +1,18 @@
 <?xml version="1.0"?>
 <!-- Main URDF including controller info -->
-<robot xmlns:xacro="http://www.ros.org/wiki/xacro" name="embla_robot">
+<robot name="embla" xmlns:xacro="http://www.ros.org/wiki/xacro">
+  <!-- Specify gazebo_control:=true to include the embla.gazebo_ros2_control.xacro instead of the
+  normal control file -->
+  <xacro:arg name="gazebo_control" default="false" />
   <!-- Base URDF -->
   <xacro:include filename="embla_description.urdf.xacro" />
-  <!-- Import ros2_control description -->
-  <xacro:include filename="$(find embla_controller)/ros2_control/embla.ros2_control.xacro" />
+  <!-- Import ros2_control description: use embla.gazebo_ros2_control.xacro if specified;
+  embla.ros2_control.xacro otherwise -->
+  <xacro:if value="$(arg gazebo_control)">
+    <xacro:include filename="$(find embla_controller)/ros2_control/embla.gazebo_ros2_control.xacro" />
+  </xacro:if>
+  <xacro:unless value="$(arg gazebo_control)">
+    <xacro:include filename="$(find embla_controller)/ros2_control/embla.ros2_control.xacro" />
+  </xacro:unless>
   <xacro:embla_ros2_control name="Embla" />
   <!-- Gazebo common -->

File: description/urdf/imu.xacro (robot description, xacro)
@@ -1,11 +1,11 @@
 <?xml version="1.0"?>
-<robot xmlns:xacro="http://www.ros.org/wiki/xacro" name="embla">
+<robot name="embla" xmlns:xacro="http://www.ros.org/wiki/xacro">
 	<!-- IMU -->
-	<xacro:property name="imuHeight" value="0.010"/>
-	<xacro:property name="imuDiameter" value="0.031"/>
-	<xacro:property name="imuMass" value="0.030"/>
+	<xacro:property name="imuHeight" value="0.010" />
+	<xacro:property name="imuDiameter" value="0.031" />
+	<xacro:property name="imuMass" value="0.030" />
 	<joint name="imu_joint" type="fixed">
-		<parent link="base_link"/>
-		<child link="imu_link"/>
+		<parent link="base_link" />
+		<child link="imu_link" />
 		<!-- Origin is at center of IMU which is placed on chassis top, a little back from midpoint -->
 		<origin xyz="-0.05 0 ${chassisHeight/2 + imuHeight/2}" rpy="0 0 ${PI/2}" />
@@ -13,20 +13,20 @@
 	<link name="imu_link">
 		<collision>
-			<origin xyz="0 0 0" rpy="0 0 0"/>
+			<origin xyz="0 0 0" rpy="0 0 0" />
 			<geometry>
-				<cylinder length="${imuHeight}" radius="${imuDiameter/2}"/>
+				<cylinder length="${imuHeight}" radius="${imuDiameter/2}" />
 			</geometry>
 		</collision>
 		<visual>
-			<origin xyz="0 0 0" rpy="0 0 0"/>
+			<origin xyz="0 0 0" rpy="0 0 0" />
 			<geometry>
-				<cylinder length="${imuHeight}" radius="${imuDiameter/2}"/>
+				<cylinder length="${imuHeight}" radius="${imuDiameter/2}" />
 			</geometry>
-			<material name="orange"/>
+			<material name="orange" />
 		</visual>
 		<inertial>
-			<origin xyz="0 0 0" rpy="0 0 0"/>
-			<mass value="${imuMass}"/>
-			<xacro:cylinder_inertia m="${imuMass}" r="${imuDiameter/2}" h="${imuHeight}"/>
+			<origin xyz="0 0 0" rpy="0 0 0" />
+			<mass value="${imuMass}" />
+			<xacro:cylinder_inertia m="${imuMass}" r="${imuDiameter/2}" h="${imuHeight}" />
 		</inertial>
 	</link>

File: description/urdf/lidar.xacro (robot description, xacro)
@@ -1,14 +1,15 @@
 <?xml version="1.0"?>
-<robot xmlns:xacro="http://www.ros.org/wiki/xacro" name="embla">
+<robot name="embla" xmlns:xacro="http://www.ros.org/wiki/xacro">
 	<!-- Lidar -->
-	<xacro:property name="lidarHeight" value="0.041"/>
-	<xacro:property name="lidarDiameter" value="0.076"/>
-	<xacro:property name="lidarMass" value="0.190"/>
+	<xacro:property name="lidarHeight" value="0.041" />
+	<xacro:property name="lidarDiameter" value="0.076" />
+	<xacro:property name="lidarMass" value="0.190" />
 	<joint name="lidar_joint" type="fixed">
-		<parent link="base_link"/>
-		<child link="lidar_link"/>
+		<parent link="base_link" />
+		<child link="lidar_link" />
 		<!--
 			Origin is at center of Lidar which is placed on chassis top, 5 cm forward of midpoint.
-			NOTE The origin has been rotated PI radians around Z because the RPLidar has X pointing backwards and Y pointing right compared to conventional robot orientation (X forward, Y left, Z up).
+			NOTE The origin has been rotated PI radians around Z because the RPLidar has X pointing backwards
+		and Y pointing right compared to conventional robot orientation (X forward, Y left, Z up).
 			This, however, will mess up the /scan data when running in Gazebo. -->
 		<origin xyz="0.04 0 ${chassisHeight/2 + lidarHeight/2}" rpy="0 0 ${PI}" />
@@ -16,23 +17,25 @@
 	<link name="lidar_link">
 		<collision>
-			<origin xyz="0 0 0" rpy="0 0 0"/>
+			<origin xyz="0 0 0" rpy="0 0 0" />
 			<geometry>
-				<cylinder length="${lidarHeight}" radius="${lidarDiameter/2}"/>
+				<cylinder length="${lidarHeight}" radius="${lidarDiameter/2}" />
 			</geometry>
 		</collision>
 		<visual>
-			<origin xyz="0 0 -${lidarHeight/2}" rpy="${PI/2} 0 ${3*PI/2}"/>
+			<origin xyz="0 0 -${lidarHeight/2}" rpy="${PI/2} 0 ${3*PI/2}" />
 			<geometry>
-				<mesh filename="package://embla_controller/urdf/meshes/rplidar.dae" scale="0.001 0.001 0.001"/>
+				<mesh filename="package://embla_controller/urdf/meshes/rplidar.dae"
+					scale="0.001 0.001 0.001" />
 			</geometry>
-			<material name="black"/>
+			<material name="black" />
 		</visual>
 		<inertial>
-			<origin xyz="0 0 0" rpy="0 0 0"/>
-			<mass value="${lidarMass}"/>
-			<xacro:cylinder_inertia m="${lidarMass}" r="${lidarDiameter/2}" h="${lidarHeight}"/>
+			<origin xyz="0 0 0" rpy="0 0 0" />
+			<mass value="${lidarMass}" />
+			<xacro:cylinder_inertia m="${lidarMass}" r="${lidarDiameter/2}" h="${lidarHeight}" />
 		</inertial>
 	</link>
-	<!-- from ROSbot 2.0 https://github.com/husarion/rosbot_description/blob/master/src/rosbot_description/urdf/rosbot.xacro -->
+	<!-- from ROSbot 2.0
+	https://github.com/husarion/rosbot_description/blob/master/src/rosbot_description/urdf/rosbot.xacro -->
 	<!-- RpLidar using GPU -->
 	<gazebo reference="lidar_link">

File: description/urdf/macros.xacro (robot description, xacro)
@@ -1,9 +1,11 @@
 <?xml version="1.0"?>
-<robot xmlns:xacro="http://www.ros.org/wiki/xacro">
+<robot name="embla" xmlns:xacro="http://www.ros.org/wiki/xacro">
 	<xacro:macro name="cylinder_inertia" params="m r h">
-		<inertia ixx="${m*(3*r*r+h*h)/12}" ixy="0" ixz="0" iyy="${m*(3*r*r+h*h)/12}" iyz="0" izz="${m*r*r/2}" />
+		<inertia ixx="${m*(3*r*r+h*h)/12}" ixy="0" ixz="0" iyy="${m*(3*r*r+h*h)/12}" iyz="0"
+			izz="${m*r*r/2}" />
 	</xacro:macro>
 	<xacro:macro name="box_inertia" params="m x y z">
-		<inertia ixx="${m*(y*y+z*z)/12}" ixy="0" ixz="0" iyy="${m*(x*x+z*z)/12}" iyz="0" izz="${m*(x*x+z*z)/12}" />
+		<inertia ixx="${m*(y*y+z*z)/12}" ixy="0" ixz="0" iyy="${m*(x*x+z*z)/12}" iyz="0"
+			izz="${m*(x*x+z*z)/12}" />
 	</xacro:macro>
 	<xacro:macro name="sphere_inertia" params="m r">

File: description/urdf/wheel.xacro (robot description, xacro)
@@ -1,4 +1,4 @@
 <?xml version="1.0"?>
-<robot xmlns:xacro="http://www.ros.org/wiki/xacro" name="embla">
+<robot name="embla" xmlns:xacro="http://www.ros.org/wiki/xacro">
 	<!-- Macro for wheels.
 	Parameters:
@@ -10,16 +10,17 @@
 	<xacro:macro name="wheel" params="lr fr tY tX">
 		<joint name="${lr}_${fr}_wheel_joint" type="continuous">
-			<parent link="base_link"/>
-			<child link="${lr}_${fr}_wheel"/>
-			<origin xyz="${tX * wheelXDistance/2} ${tY * wheelYDistance/2} ${-chassisHeight/2 - (chassisGroundClearance - wheelRadius)}"/>
-			<axis xyz="0 1 0" rpy="0 0 0"/>
-			<limit effort="100" velocity="100"/>
-			<joint_properties damping="0.0" friction="0.5"/>
+			<parent link="base_link" />
+			<child link="${lr}_${fr}_wheel" />
+			<origin
+				xyz="${tX * wheelXDistance/2} ${tY * wheelYDistance/2} ${-chassisHeight/2 - (chassisGroundClearance - wheelRadius)}" />
+			<axis xyz="0 1 0" rpy="0 0 0" />
+			<limit effort="100" velocity="100" />
+			<joint_properties damping="0.0" friction="0.5" />
 		</joint>
 		<link name="${lr}_${fr}_wheel">
 			<collision>
-				<origin xyz="0 0 0" rpy="${PI/2} 0 0"/>
+				<origin xyz="0 0 0" rpy="${PI/2} 0 0" />
 				<geometry>
-					<cylinder length="${wheelWidth}" radius="${wheelRadius}"/>
+					<cylinder length="${wheelWidth}" radius="${wheelRadius}" />
 				</geometry>
 				<surface>
@@ -33,14 +34,14 @@
 			</collision>
 			<visual>
-				<origin xyz="0 0 0" rpy="${PI/2} 0 0"/>
+				<origin xyz="0 0 0" rpy="${PI/2} 0 0" />
 				<geometry>
-					<cylinder length="${wheelWidth}" radius="${wheelRadius}"/>
+					<cylinder length="${wheelWidth}" radius="${wheelRadius}" />
 				</geometry>
-				<material name="black"/>
+				<material name="black" />
 			</visual>
 			<inertial>
-				<origin xyz="0 0 0" rpy="${PI/2} 0 0"/>
-				<mass value="${wheelMass}"/>
-				<xacro:cylinder_inertia m="${wheelMass}" r="${wheelRadius}" h="${wheelWidth}"/>
+				<origin xyz="0 0 0" rpy="${PI/2} 0 0" />
+				<mass value="${wheelMass}" />
+				<xacro:cylinder_inertia m="${wheelMass}" r="${wheelRadius}" h="${wheelWidth}" />
 			</inertial>
 		</link>
